File: schematics/funklicht.sch (EAGLE design)
At the start: 23 parts, among them IC2 5V, SW1 push, SW2 push, SW3 push, SW4 push

Commit message: schematics done
Parts:
- removed U$3: TRANSMITTER, funkmodule:TRANSMITTER
- added 3.3V: LM3940, voltage_regulator:LM3940
- added C5, C6: 100uF, rcl:CPOL-EUTT2D6
- added HC-SR04: (no value), con-lstb:MA04-1
- added SV2: (no value), con-lstb:MA06-1
- added U$4: NRF24L01, funkmodule:NRF24L01
- C1, C2, C3, C4: device rcl:C-EU050-025X075 -> rcl:C-EU025-024X044
- LED1: value RGB -> (none)
- U$2: value RECIEVER -> AB5V; device funkmodule:RECIEVER -> power_supply:AB5V
Connections:
- removed net TX_ENABLE: U$1.D7, U$3.TX_ENABLE
- removed net VDD: IC2.OUT, LED1.VCC, R4.2, R5.2, R6.2, R7.2, U$1.VIN, U$2.VDD
- new net N$10: U$1.D8, U$4.CE
- new net N$11: R3.1, SV2.4, U$1.D5
- new net N$12: R1.1, SV2.3, U$1.D3
- new net N$13: HC-SR04.3, U$1.D2
- new net N$14: HC-SR04.2, U$1.D4
- new net N$21: SV2.1, U$1.D7
- new net N$22: SV2.2, U$1.A5
- new net N$8: U$1.D11, U$4.MOSI
- new net N$9: U$1.D10, U$4.CSN
- new net VCC: 3.3V.IN, C6.+, HC-SR04.1, IC2.OUT, R4.2, R5.2, R6.2, R7.2, U$1.VIN, U$2.+
- net GND: now also 3.3V.GND, C5.-, C6.-, HC-SR04.4, LED1.GND, SV2.6, U$2.-, U$4.GND; no longer U$2.GND, U$3.GND
- net N$1: now also U$1.A0; no longer U$1.D2
- net N$15: now also U$1.A1; no longer U$1.D4
- net N$16: now also U$1.A2; no longer U$1.D5
- net N$17: now also U$1.A3; no longer U$1.D6
- net N$18: no longer U$1.D8
- net N$2: now also R2.1, SV2.5, U$1.D6; no longer U$1.D3, U$3.DATA
- net N$3: now also U$4.MISO; no longer U$2.DATA
- net N$4: now also 3.3V.OUT, C5.+, U$4.VCC; no longer R1.1, U$1.D11
- net N$5: now also U$1.D9, U$4.IRQ; no longer R3.1, U$1.D10
- net N$6: now also U$1.D13, U$4.SCK; no longer R2.1, U$1.D9
Other:
- moved on the sheet: BUZZER, C1, C2, C3, C4, G1, LED1, R1, R2, R3, R4, R5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

Commit message: hand routed board
Parts:
- SV2: device con-lstb:MA06-1 -> con-lstb:MA07-1
- renumbered U$4 to U$3
Connections:
- removed net N$4: 3.3V.OUT, C5.+, U$3.VCC
- net GND: now also SV2.7; no longer SV2.6
- net N$12: now also SV2.6; no longer SV2.3
- net N$18: now also U$1.A4
- net N$20: now also SV2.1
- net N$21: now also SV2.2; no longer SV2.1
- net N$22: now also SV2.3; no longer SV2.2
- net VCC: now also 3.3V.OUT, C5.+, U$3.VCC
Other:
- moved on the sheet: 3.3V

Commit message: fertiges platinenlayout
Parts:
- renumbered SV2 to 9V
Connections:
- new net 3V3: 3.3V.OUT, C5.+, U$3.3V3
- net N$15: no longer SW1.S
- net VCC: no longer 3.3V.OUT, C5.+, U$3.VCC
Changed lines of the file:
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@@
 <part name="HC-SR04" library="con-lstb" deviceset="MA04-1" device=""/>
 <part name="GND12" library="supply1" deviceset="GND" device=""/>
-<part name="SV2" library="con-lstb" deviceset="MA07-1" device=""/>
+<part name="9V" library="con-lstb" deviceset="MA07-1" device=""/>
 <part name="U$3" library="funkmodule" deviceset="NRF24L01" device=""/>
 </parts>
@@
 <instance part="HC-SR04" gate="1" x="93.98" y="134.62" rot="R270"/>
 <instance part="GND12" gate="1" x="96.52" y="121.92"/>
-<instance part="SV2" gate="1" x="134.62" y="157.48" rot="R180"/>
+<instance part="9V" gate="1" x="134.62" y="157.48" rot="R180"/>
 <instance part="U$3" gate="G$1" x="180.34" y="78.74"/>
 </instances>
@@
 <pinref part="GND11" gate="1" pin="GND"/>
 <wire x1="124.46" y1="147.32" x2="124.46" y2="149.86" width="0.1524" layer="91"/>
-<pinref part="SV2" gate="1" pin="7"/>
+<pinref part="9V" gate="1" pin="7"/>
 <wire x1="124.46" y1="149.86" x2="127" y2="149.86" width="0.1524" layer="91"/>
 </segment>
@@
 <segment>
 <pinref part="R5" gate="G$1" pin="1"/>
-<pinref part="SW1" gate="1" pin="S"/>
-<wire x1="162.56" y1="40.64" x2="162.56" y2="38.1" width="0.1524" layer="91"/>
 <wire x1="162.56" y1="40.64" x2="152.4" y2="40.64" width="0.1524" layer="91"/>
 <wire x1="152.4" y1="40.64" x2="152.4" y2="12.7" width="0.1524" layer="91"/>
 <wire x1="152.4" y1="12.7" x2="116.84" y2="12.7" width="0.1524" layer="91"/>
-<junction x="162.56" y="40.64"/>
-<pinref part="SW1" gate="1" pin="S1"/>
 <pinref part="C3" gate="G$1" pin="1"/>
-<wire x1="165.1" y1="38.1" x2="167.64" y2="38.1" width="0.1524" layer="91"/>
-<wire x1="162.56" y1="40.64" x2="167.64" y2="40.64" width="0.1524" layer="91"/>
+<wire x1="162.56" y1="40.64" x2="165.1" y2="40.64" width="0.1524" layer="91"/>
+<wire x1="165.1" y1="40.64" x2="167.64" y2="40.64" width="0.1524" layer="91"/>
 <wire x1="167.64" y1="40.64" x2="167.64" y2="38.1" width="0.1524" layer="91"/>
-<junction x="167.64" y="38.1"/>
 <wire x1="116.84" y1="12.7" x2="116.84" y2="63.5" width="0.1524" layer="91"/>
 <pinref part="U$1" gate="G$1" pin="A1"/>
 <wire x1="116.84" y1="63.5" x2="104.14" y2="63.5" width="0.1524" layer="91"/>
+<pinref part="SW1" gate="1" pin="S1"/>
+<wire x1="165.1" y1="38.1" x2="165.1" y2="40.64" width="0.1524" layer="91"/>
+<junction x="165.1" y="40.64"/>
+<junction x="162.56" y="40.64"/>
 </segment>
 </net>
@@
 <wire x1="12.7" y1="66.04" x2="25.4" y2="66.04" width="0.1524" layer="91"/>
 <pinref part="IC2" gate="1" pin="IN"/>
-<pinref part="SV2" gate="1" pin="1"/>
+<pinref part="9V" gate="1" pin="1"/>
 <wire x1="127" y1="165.1" x2="12.7" y2="165.1" width="0.1524" layer="91"/>
 <wire x1="12.7" y1="165.1" x2="12.7" y2="66.04" width="0.1524" layer="91"/>
+<junction x="12.7" y="66.04"/>
 </segment>
 </net>
@@
 <junction x="190.5" y="106.68"/>
 </segment>
-<segment>
-<pinref part="U$3" gate="G$1" pin="VCC"/>
-<wire x1="167.64" y1="73.66" x2="162.56" y2="73.66" width="0.1524" layer="91"/>
-<wire x1="162.56" y1="73.66" x2="162.56" y2="106.68" width="0.1524" layer="91"/>
-<pinref part="3.3V" gate="G$1" pin="OUT"/>
-<pinref part="C5" gate="G$1" pin="+"/>
-<wire x1="170.18" y1="106.68" x2="167.64" y2="106.68" width="0.1524" layer="91"/>
-<wire x1="167.64" y1="106.68" x2="167.64" y2="104.14" width="0.1524" layer="91"/>
-<wire x1="162.56" y1="106.68" x2="167.64" y2="106.68" width="0.1524" layer="91"/>
-<junction x="167.64" y="106.68"/>
-</segment>
 </net>
 <net name="N$5" class="0">
@@
 <wire x1="116.84" y1="154.94" x2="116.84" y2="119.38" width="0.1524" layer="91"/>
 <junction x="116.84" y="119.38"/>
-<pinref part="SV2" gate="1" pin="5"/>
+<pinref part="9V" gate="1" pin="5"/>
 <wire x1="116.84" y1="154.94" x2="127" y2="154.94" width="0.1524" layer="91"/>
 </segment>
@@
 <wire x1="114.3" y1="157.48" x2="114.3" y2="127" width="0.1524" layer="91"/>
 <junction x="114.3" y="127"/>
-<pinref part="SV2" gate="1" pin="4"/>
+<pinref part="9V" gate="1" pin="4"/>
 <wire x1="127" y1="157.48" x2="114.3" y2="157.48" width="0.1524" layer="91"/>
 </segment>
@@
 <wire x1="111.76" y1="96.52" x2="104.14" y2="96.52" width="0.1524" layer="91"/>
 <junction x="111.76" y="134.62"/>
-<pinref part="SV2" gate="1" pin="6"/>
+<pinref part="9V" gate="1" pin="6"/>
 <wire x1="111.76" y1="152.4" x2="111.76" y2="134.62" width="0.1524" layer="91"/>
 <wire x1="127" y1="152.4" x2="111.76" y2="152.4" width="0.1524" layer="91"/>
@@
 <wire x1="104.14" y1="86.36" x2="119.38" y2="86.36" width="0.1524" layer="91"/>
 <wire x1="119.38" y1="86.36" x2="119.38" y2="162.56" width="0.1524" layer="91"/>
-<pinref part="SV2" gate="1" pin="2"/>
+<pinref part="9V" gate="1" pin="2"/>
 <wire x1="127" y1="162.56" x2="119.38" y2="162.56" width="0.1524" layer="91"/>
 </segment>
@@
 <wire x1="104.14" y1="53.34" x2="121.92" y2="53.34" width="0.1524" layer="91"/>
 <wire x1="121.92" y1="53.34" x2="121.92" y2="160.02" width="0.1524" layer="91"/>
-<pinref part="SV2" gate="1" pin="3"/>
+<pinref part="9V" gate="1" pin="3"/>
 <wire x1="127" y1="160.02" x2="121.92" y2="160.02" width="0.1524" layer="91"/>
 </segment>
@@
 </segment>
 </net>
+<net name="3V3" class="0">
+<segment>
+<pinref part="U$3" gate="G$1" pin="3V3"/>
+<wire x1="167.64" y1="73.66" x2="162.56" y2="73.66" width="0.1524" layer="91"/>
+<wire x1="162.56" y1="73.66" x2="162.56" y2="106.68" width="0.1524" layer="91"/>
+<pinref part="C5" gate="G$1" pin="+"/>
+<pinref part="3.3V" gate="G$1" pin="OUT"/>
+<wire x1="170.18" y1="106.68" x2="167.64" y2="106.68" width="0.1524" layer="91"/>
+<wire x1="167.64" y1="106.68" x2="167.64" y2="104.14" width="0.1524" layer="91"/>
+<wire x1="162.56" y1="106.68" x2="167.64" y2="106.68" width="0.1524" layer="91"/>
+<junction x="167.64" y="106.68"/>
+</segment>
+</net>
